File: v2_pcb/leds.kicad_sch (KiCad schematic)
At the start: 71 parts

Commit message: work
Parts:
- removed C13, C28, C29, C30: 100nF, symbol Device:C
- added C16, C17, C18: 4.7μF, Capacitor_SMD:C_1206_3216Metric_Pad1.33x1.80mm_HandSolder, symbol Device:C
- added C34, C35, C36, C37, C38, C39, C40, C41, C42, C43, C44, C45, C46, C47, C48, C49, C50, C51, C52, C53: 1μF, Capacitor_SMD:C_1206_3216Metric_Pad1.33x1.80mm_HandSolder, symbol Device:C
- added C54, C55, C56, C57, C58, C59, C60, C61, C62, C63, C64, C65, C66, C67, C68, C69, C70, C71, C72, C73, C74, C75, C76, C77, C78, C79, C80, C81, C82, C83, C84, C85, C86, C87, C88, C89, C90, C91, C92, C93, C94, C95, C96: 100nF, Capacitor_SMD:C_1206_3216Metric_Pad1.33x1.80mm_HandSolder, symbol Device:C
- C11, C12, C19, C20, C21, C22, C23, C24, C25, C26: value 100nF -> 4.7μF; footprint (none) -> Capacitor_SMD:C_1206_3216Metric_Pad1.33x1.80mm_HandSolder; Manufacturer Part Number (none) -> CL31B475KAHNNNE; Vendor (none) -> Digi-Key; Vendor Part Number (none) -> 1276-1055-1-ND
- C13: renamed from C10; value 1μF -> 4.7μF; footprint (none) -> Capacitor_SMD:C_1206_3216Metric_Pad1.33x1.80mm_HandSolder; Manufacturer Part Number (none) -> CL31B475KAHNNNE; Vendor (none) -> Digi-Key; Vendor Part Number (none) -> 1276-1055-1-ND
- C14, C15: value 1μF -> 4.7μF; footprint (none) -> Capacitor_SMD:C_1206_3216Metric_Pad1.33x1.80mm_HandSolder; Manufacturer Part Number (none) -> CL31B475KAHNNNE; Vendor (none) -> Digi-Key; Vendor Part Number (none) -> 1276-1055-1-ND
- C27, C31, C32, C33: value 100nF -> 1μF; footprint (none) -> Capacitor_SMD:C_1206_3216Metric_Pad1.33x1.80mm_HandSolder; Manufacturer Part Number (none) -> CL31B105KAHNNNE; Vendor (none) -> Digi-Key; Vendor Part Number (none) -> 1276-1097-1-ND
- C28: renamed from C16; footprint (none) -> Capacitor_SMD:C_1206_3216Metric_Pad1.33x1.80mm_HandSolder; Manufacturer Part Number (none) -> CL31B105KAHNNNE; Vendor (none) -> Digi-Key; Vendor Part Number (none) -> 1276-1097-1-ND
- C29: renamed from C17; footprint (none) -> Capacitor_SMD:C_1206_3216Metric_Pad1.33x1.80mm_HandSolder; Manufacturer Part Number (none) -> CL31B105KAHNNNE; Vendor (none) -> Digi-Key; Vendor Part Number (none) -> 1276-1097-1-ND
- C30: renamed from C18; footprint (none) -> Capacitor_SMD:C_1206_3216Metric_Pad1.33x1.80mm_HandSolder; Manufacturer Part Number (none) -> CL31B105KAHNNNE; Vendor (none) -> Digi-Key; Vendor Part Number (none) -> 1276-1097-1-ND
- D1, D10, D11, D12, D13, D14, D15, D16, D17, D18, D19, D2, D20, D21, D22, D3, D4, D47, D5, D6, D7, D8, D9: Manufacturer Part Number (none) -> IN-PI554FCH; Vendor (none) -> Digi-Key; Vendor Part Number (none) -> 1830-1106-1-ND
- D23: renamed from D45; Manufacturer Part Number (none) -> IN-PI554FCH; Vendor (none) -> Digi-Key; Vendor Part Number (none) -> 1830-1106-1-ND
- D24: renamed from D23; Manufacturer Part Number (none) -> IN-PI554FCH; Vendor (none) -> Digi-Key; Vendor Part Number (none) -> 1830-1106-1-ND
- D25: renamed from D24; Manufacturer Part Number (none) -> IN-PI554FCH; Vendor (none) -> Digi-Key; Vendor Part Number (none) -> 1830-1106-1-ND
- D26: renamed from D25; Manufacturer Part Number (none) -> IN-PI554FCH; Vendor (none) -> Digi-Key; Vendor Part Number (none) -> 1830-1106-1-ND
- D27: renamed from D26; Manufacturer Part Number (none) -> IN-PI554FCH; Vendor (none) -> Digi-Key; Vendor Part Number (none) -> 1830-1106-1-ND
- D28: renamed from D27; Manufacturer Part Number (none) -> IN-PI554FCH; Vendor (none) -> Digi-Key; Vendor Part Number (none) -> 1830-1106-1-ND
- D29: renamed from D28; Manufacturer Part Number (none) -> IN-PI554FCH; Vendor (none) -> Digi-Key; Vendor Part Number (none) -> 1830-1106-1-ND
- D30: renamed from D29; Manufacturer Part Number (none) -> IN-PI554FCH; Vendor (none) -> Digi-Key; Vendor Part Number (none) -> 1830-1106-1-ND
- D31: renamed from D30; Manufacturer Part Number (none) -> IN-PI554FCH; Vendor (none) -> Digi-Key; Vendor Part Number (none) -> 1830-1106-1-ND
- D32: renamed from D31; Manufacturer Part Number (none) -> IN-PI554FCH; Vendor (none) -> Digi-Key; Vendor Part Number (none) -> 1830-1106-1-ND
- D33: renamed from D32; Manufacturer Part Number (none) -> IN-PI554FCH; Vendor (none) -> Digi-Key; Vendor Part Number (none) -> 1830-1106-1-ND
- D34: renamed from D33; Manufacturer Part Number (none) -> IN-PI554FCH; Vendor (none) -> Digi-Key; Vendor Part Number (none) -> 1830-1106-1-ND
- D35: renamed from D46; Manufacturer Part Number (none) -> IN-PI554FCH; Vendor (none) -> Digi-Key; Vendor Part Number (none) -> 1830-1106-1-ND
- D36: renamed from D34; Manufacturer Part Number (none) -> IN-PI554FCH; Vendor (none) -> Digi-Key; Vendor Part Number (none) -> 1830-1106-1-ND
- D37: renamed from D35; Manufacturer Part Number (none) -> IN-PI554FCH; Vendor (none) -> Digi-Key; Vendor Part Number (none) -> 1830-1106-1-ND
- D38: renamed from D36; Manufacturer Part Number (none) -> IN-PI554FCH; Vendor (none) -> Digi-Key; Vendor Part Number (none) -> 1830-1106-1-ND
- D39: renamed from D37; Manufacturer Part Number (none) -> IN-PI554FCH; Vendor (none) -> Digi-Key; Vendor Part Number (none) -> 1830-1106-1-ND
- D40: renamed from D38; Manufacturer Part Number (none) -> IN-PI554FCH; Vendor (none) -> Digi-Key; Vendor Part Number (none) -> 1830-1106-1-ND
- D41: renamed from D39; Manufacturer Part Number (none) -> IN-PI554FCH; Vendor (none) -> Digi-Key; Vendor Part Number (none) -> 1830-1106-1-ND
- D42: renamed from D40; Manufacturer Part Number (none) -> IN-PI554FCH; Vendor (none) -> Digi-Key; Vendor Part Number (none) -> 1830-1106-1-ND
- D43: renamed from D41; Manufacturer Part Number (none) -> IN-PI554FCH; Vendor (none) -> Digi-Key; Vendor Part Number (none) -> 1830-1106-1-ND
- D44: renamed from D42; Manufacturer Part Number (none) -> IN-PI554FCH; Vendor (none) -> Digi-Key; Vendor Part Number (none) -> 1830-1106-1-ND
- D45: renamed from D43; Manufacturer Part Number (none) -> IN-PI554FCH; Vendor (none) -> Digi-Key; Vendor Part Number (none) -> 1830-1106-1-ND
- D46: renamed from D44; Manufacturer Part Number (none) -> IN-PI554FCH; Vendor (none) -> Digi-Key; Vendor Part Number (none) -> 1830-1106-1-ND
Connections:
- net +5V: now also C16.1, C17.1, C18.1, C34.1, C35.1, C36.1, C37.1, C38.1, C39.1, C40.1, C41.1, C42.1, C43.1, C44.1, C45.1, C46.1, C47.1, C48.1, C49.1, C50.1, C51.1, C52.1, C53.1, C54.1, C55.1, C56.1, C57.1, C58.1, C59.1, C60.1, C61.1, C62.1, C63.1, C64.1, C65.1, C66.1, C67.1, C68.1, C69.1, C70.1, C71.1, C72.1, C73.1, C74.1, C75.1, C76.1, C77.1, C78.1, C79.1, C80.1, C81.1, C82.1, C83.1, C84.1, C85.1, C86.1, C87.1, C88.1, C89.1, C90.1, C91.1, C92.1, C93.1, C94.1, C95.1, C96.1
- net GND: now also C16.2, C17.2, C18.2, C34.2, C35.2, C36.2, C37.2, C38.2, C39.2, C40.2, C41.2, C42.2, C43.2, C44.2, C45.2, C46.2, C47.2, C48.2, C49.2, C50.2, C51.2, C52.2, C53.2, C54.2, C55.2, C56.2, C57.2, C58.2, C59.2, C60.2, C61.2, C62.2, C63.2, C64.2, C65.2, C66.2, C67.2, C68.2, C69.2, C70.2, C71.2, C72.2, C73.2, C74.2, C75.2, C76.2, C77.2, C78.2, C79.2, C80.2, C81.2, C82.2, C83.2, C84.2, C85.2, C86.2, C87.2, C88.2, C89.2, C90.2, C91.2, C92.2, C93.2, C94.2, C95.2, C96.2
Other:
- moved on the sheet: C13, C14, C28, C29, C30, D1, D10, D11, D12, D13, D14, D15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
