File: v2_pcb/ieee-sign.kicad_sch (KiCad schematic)
At the start: 0 parts

Commit message: schematic
Parts:
- added C1, C8: 1μF, symbol Device:C
- added C2, C3, C4, C7: 100nF, symbol Device:C
- added C5, C6: 20pF, symbol Device:C
- added C9: 10μF, symbol Device:C
- added J1: AVR-ISP-6, symbol Connector:AVR-ISP-6
- added J2: USB_C_Receptacle, symbol Connector:USB_C_Receptacle
- added JP1, JP2: (no value), symbol Jumper:SolderJumper_2_Open
- added R1: 10kΩ, symbol Device:R_US
- added R2, R3: 5.1kΩ, symbol Device:R_US
- added R4, R6, R8, R9: 1.5kΩ, symbol Device:R_US
- added R5, R7: 8.2kΩ, symbol Device:R_US
- added SW1, SW2: SW_Push, Button_Switch_THT:SW_PUSH_6mm, symbol Switch:SW_Push
- added TP1, TP2, TP3, TP4, TP5: TestPoint, symbol Connector:TestPoint
- added U1: ATmega32U2-A, Package_QFP:TQFP-32_7x7mm_P0.8mm, symbol MCU_Microchip_ATmega:ATmega32U2-A
- added U2: LP2901D, Package_SO:SOIC-14_3.9x8.7mm_P1.27mm, symbol Comparator:LP2901D
- added Y1: Crystal, symbol Device:Crystal
Connections:
- new net: R4.1, R5.2, U2.4 (-)
- new net: R7.2, R8.1, U2.10 (-)
- new net: C1.1, U1.27 (UCAP)
- new net: C6.1, U1.1 (XTAL1), Y1.1
- new net: JP1.1 (A), U1.19 (PB5)
- new net: C5.1, U1.2 (PC0/XTAL2), Y1.2
- new net: JP2.1 (A), U1.6 (PD0)
- new net: R8.2, R9.1, U2.8 (-)
- new net: R4.2, R6.1, U2.6 (-)
- new net: JP1.2 (B), JP2.2 (B), SW2.2
- new net +5V: C2.1, C3.1, C4.1, C8.1, C9.1, J1.2 (VCC), J2.A4 (VBUS), J2.A9 (VBUS), J2.B4 (VBUS), J2.B9 (VBUS), R1.1, R5.1, R7.1, TP2.1, U1.31 (UVCC), U1.32 (AVCC), U1.4 (VCC), U2.3 (V+)
- new net CC1: J2.A5 (CC1), R2.1, TP4.1, U2.5 (+), U2.7 (+)
- new net CC1_H: U1.5 (PC2), U2.2
- new net CC1_L: U1.26 (PC4), U2.1
- new net CC2: J2.B5 (CC2), R3.1, TP5.1, U2.11 (+), U2.9 (+)
- new net CC2_H: U1.25 (PC5), U2.13
- new net CC2_L: U1.23 (PC6), U2.14
- new net D+: J2.A6 (D+), J2.B6 (D+), U1.29 (D+)
- new net D-: J2.A7 (D-), J2.B7 (D-), U1.30 (D-)
- new net GND: C1.2, C2.2, C3.2, C4.2, C5.2, C6.2, C7.2, C8.2, C9.2, J1.6 (GND), J2.A1 (GND), J2.A12 (GND), J2.B1 (GND), J2.B12 (GND), J2.SH (SHIELD), R2.2, R3.2, R6.2, R9.2, SW1.1, SW2.1, TP3.1, U1.28 (UGND), U1.3 (GND), U2.12 (V-)
- new net LED: TP1.1, U1.20 (PB6)
- new net PGMR_MISO: J1.1 (MISO), U1.17 (PB3)
- new net PGMR_MOSI: J1.4 (MOSI), U1.16 (PB2)
- new net PGMR_SCK: J1.3 (SCK), U1.15 (PB1)
- new net ~{RESET}: C7.1, J1.5 (~{RST}), R1.2, SW1.2, U1.24 (PC1/~{RESET})
- no-connect marks 0 -> 21
Other:
- added sheet LEDs (leds.kicad_sch)
- company: (none) -> University of California, Santa Barbara IEEE Student Branch
- title: (none) -> IEEE Sign

Commit message: work
Parts:
- removed J2: USB_C_Receptacle, symbol Connector:USB_C_Receptacle
- added C10: 100nF, Capacitor_SMD:C_1206_3216Metric_Pad1.33x1.80mm_HandSolder, symbol Device:C
- added H1, H2, H3, H4: MountingHole, MountingHole:MountingHole_3.2mm_M3, symbol Mechanical:MountingHole
- added J2: USB_C_Receptacle, Connector_USB:USB_C_Receptacle_GCT_USB4105-xx-A_16P_TopMnt_Horizontal, symbol Connector:USB_C_Receptacle_USB2.0_16P
- added LG1: UCSB IEEE Logo, Footprints:UCSB_IEEE_Logo, symbol symbols:LOGO
- C1: renamed from C8; footprint (none) -> Capacitor_SMD:C_1206_3216Metric_Pad1.33x1.80mm_HandSolder; Manufacturer Part Number (none) -> CL31B105KAHNNNE; Vendor (none) -> Digi-Key; Vendor Part Number (none) -> 1276-1097-1-ND
- C2, C3, C4: footprint (none) -> Capacitor_SMD:C_1206_3216Metric_Pad1.33x1.80mm_HandSolder; Manufacturer Part Number (none) -> C1206C104K5RACTU; Vendor (none) -> Digi-Key; Vendor Part Number (none) -> 399-C1206C104K5RACTUCT-ND
- C5: renamed from C7; footprint (none) -> Capacitor_SMD:C_1206_3216Metric_Pad1.33x1.80mm_HandSolder; Manufacturer Part Number (none) -> C1206C104K5RACTU; Vendor (none) -> Digi-Key; Vendor Part Number (none) -> 399-C1206C104K5RACTUCT-ND
- C6: renamed from C9; footprint (none) -> Capacitor_SMD:C_1206_3216Metric_Pad1.33x1.80mm_HandSolder; Manufacturer Part Number (none) -> CL31A106MAHNNNE; Vendor (none) -> Digi-Key; Vendor Part Number (none) -> 1276-1181-1-ND
- C7: renamed from C6; footprint (none) -> Capacitor_SMD:C_0603_1608Metric_Pad1.08x0.95mm_HandSolder; Manufacturer Part Number (none) -> C0603C200J5GACTU; Vendor (none) -> Digi-Key; Vendor Part Number (none) -> 399-C0603C200J5GACTUCT-ND
- C8: renamed from C5; footprint (none) -> Capacitor_SMD:C_0603_1608Metric_Pad1.08x0.95mm_HandSolder; Manufacturer Part Number (none) -> C0603C200J5GACTU; Vendor (none) -> Digi-Key; Vendor Part Number (none) -> 399-C0603C200J5GACTUCT-ND
- C9: renamed from C1; footprint (none) -> Capacitor_SMD:C_1206_3216Metric_Pad1.33x1.80mm_HandSolder; Manufacturer Part Number (none) -> CL31B105KAHNNNE; Vendor (none) -> Digi-Key; Vendor Part Number (none) -> 1276-1097-1-ND
- J1: footprint (none) -> Connector_IDC:IDC-Header_2x03_P2.54mm_Vertical; Manufacturer Part Number (none) -> 61200621621; Vendor (none) -> Digi-Key; Vendor Part Number (none) -> 732-5394-ND
- JP1, JP2: footprint (none) -> Jumper:SolderJumper-2_P1.3mm_Open_RoundedPad1.0x1.5mm
- R1: footprint (none) -> Resistor_SMD:R_1206_3216Metric_Pad1.30x1.75mm_HandSolder; Manufacturer Part Number (none) -> RMCF1206FT10K0; Vendor (none) -> Digi-Key; Vendor Part Number (none) -> RMCF1206FT10K0CT-ND
- R2, R3: footprint (none) -> Resistor_SMD:R_1206_3216Metric_Pad1.30x1.75mm_HandSolder; Manufacturer Part Number (none) -> RC1206FR-075K1L; Vendor (none) -> Digi-Key; Vendor Part Number (none) -> 311-5.10KFRCT-ND
- R4: renamed from R5; footprint (none) -> Resistor_SMD:R_1206_3216Metric_Pad1.30x1.75mm_HandSolder; Manufacturer Part Number (none) -> RC1206FR-078K2L; Vendor (none) -> Digi-Key; Vendor Part Number (none) -> 311-8.20KFRCT-ND
- R5: renamed from R4; footprint (none) -> Resistor_SMD:R_1206_3216Metric_Pad1.30x1.75mm_HandSolder; Manufacturer Part Number (none) -> RNCP1206FTD1K50; Vendor (none) -> Digi-Key; Vendor Part Number (none) -> RNCP1206FTD1K50CT-ND
- R6, R8, R9: footprint (none) -> Resistor_SMD:R_1206_3216Metric_Pad1.30x1.75mm_HandSolder; Manufacturer Part Number (none) -> RNCP1206FTD1K50; Vendor (none) -> Digi-Key; Vendor Part Number (none) -> RNCP1206FTD1K50CT-ND
- R7: footprint (none) -> Resistor_SMD:R_1206_3216Metric_Pad1.30x1.75mm_HandSolder; Manufacturer Part Number (none) -> RC1206FR-078K2L; Vendor (none) -> Digi-Key; Vendor Part Number (none) -> 311-8.20KFRCT-ND
- SW1, SW2: Manufacturer Part Number (none) -> PTS645SL43-2 LFS; Vendor (none) -> Digi-Key; Vendor Part Number (none) -> CKN9098-ND
- TP1: renamed from TP2; footprint (none) -> TestPoint:TestPoint_Pad_D1.0mm; now left out of the parts list
- TP2: renamed from TP3; footprint (none) -> TestPoint:TestPoint_Pad_D1.0mm; now left out of the parts list
- TP3: renamed from TP4; footprint (none) -> TestPoint:TestPoint_Pad_D1.0mm; now left out of the parts list
- TP4: renamed from TP5; footprint (none) -> TestPoint:TestPoint_Pad_D1.0mm; now left out of the parts list
- TP5: renamed from TP1; footprint (none) -> TestPoint:TestPoint_Pad_D1.0mm; now left out of the parts list
- U1: Manufacturer Part Number (none) -> ATMEGA32U2-AUR; Vendor (none) -> Digi-Key; Vendor Part Number (none) -> ATMEGA32U2-AURCT-ND
- U2: Manufacturer Part Number (none) -> LP2901D; Vendor (none) -> Digi-Key; Vendor Part Number (none) -> 296-9574-5-ND
- Y1: value Crystal -> 16MHz; footprint (none) -> Crystal:Crystal_HC49-U_Vertical; Manufacturer Part Number (none) -> 16M20P2/49US; Vendor (none) -> Digi-Key; Vendor Part Number (none) -> 3155-16M20P2/49US-ND
Connections:
- net +5V: now also C10.1, J2.A4 (VBUS), J2.A9 (VBUS), J2.B4 (VBUS), J2.B9 (VBUS)
- net CC1: now also J2.A5 (CC1)
- net CC2: now also J2.B5 (CC2)
- net D+: now also J2.A6 (D+), J2.B6 (D+)
- net D-: now also J2.A7 (D-), J2.B7 (D-)
- net GND: now also C10.2, J2.A1 (GND), J2.A12 (GND), J2.B1 (GND), J2.B12 (GND), J2.SH (SHIELD)
- no-connect marks 21 -> 13

Commit message: w
Parts:
- added LG2: UCSB IEEE Logo, Footprints:UCSB_IEEE_Logo_Text, symbol symbols:LOGO
Changed lines of the file:
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@@
+	)
+	(symbol
+		(lib_id "symbols:LOGO")
+		(at 144.78 233.68 0)
+		(unit 1)
+		(body_style 1)
+		(exclude_from_sim no)
+		(in_bom no)
+		(on_board yes)
+		(in_pos_files yes)
+		(dnp no)
+		(fields_autoplaced yes)
+		(property "Reference" "LG2"
+			(at 148.59 232.4099 0)
+			(show_name no)
+			(do_not_autoplace no)
+			(effects
+				(font
+					(size 1.27 1.27)
+				)
+				(justify left)
+			)
+		)
+		(property "Value" "UCSB IEEE Logo"
+			(at 148.59 234.9499 0)
+			(show_name no)
+			(do_not_autoplace no)
+			(effects
+				(font
+					(size 1.27 1.27)
+				)
+				(justify left)
+			)
+		)
+		(property "Footprint" "Footprints:UCSB_IEEE_Logo_Text"
+			(at 144.78 233.68 0)
+			(hide yes)
+			(show_name no)
+			(do_not_autoplace no)
+			(effects
+				(font
+					(size 1.27 1.27)
+				)
+			)
+		)
+		(property "Datasheet" ""
+			(at 144.78 233.68 0)
+			(hide yes)
+			(show_name no)
+			(do_not_autoplace no)
+			(effects
+				(font
+					(size 1.27 1.27)
+				)
+			)
+		)
+		(property "Description" ""
+			(at 144.78 233.68 0)
+			(hide yes)
+			(show_name no)
+			(do_not_autoplace no)
+			(effects
+				(font
+					(size 1.27 1.27)
+				)
+			)
+		)
+		(property "Manufacturer Part Number" ""
+			(at 144.78 233.68 0)
+			(hide yes)
+			(show_name no)
+			(do_not_autoplace no)
+			(effects
+				(font
+					(size 1.27 1.27)
+				)
+			)
+		)
+		(property "Vendor" ""
+			(at 144.78 233.68 0)
+			(hide yes)
+			(show_name no)
+			(do_not_autoplace no)
+			(effects
+				(font
+					(size 1.27 1.27)
+				)
+			)
+		)
+		(property "Vendor Part Number" ""
+			(at 144.78 233.68 0)
+			(hide yes)
+			(show_name no)
+			(do_not_autoplace no)
+			(effects
+				(font
+					(size 1.27 1.27)
+				)
+			)
+		)
+		(instances
+			(project "ieee-sign"
+				(path "/13ce365d-1ebc-4b37-b0cf-a22bb69a2d67"
+					(reference "LG2")
+					(unit 1)
+				)
+			)
+		)
 	)
 	(symbol
