File: v2_pcb/ieee-sign.kicad_pcb (KiCad board)
At the start: 2 copper layers, 330 x 130 mm, 171 parts, among them J1 AVR-ISP-6, J2 USB_C_Receptacle, SW1 SW_Push, SW2 SW_Push, U1 ATmega32U2-A, U2 LP2901D, Y1 16MHz

Commit message: w
Parts:
- added LG2: UCSB IEEE Logo, Footprints:UCSB_IEEE_Logo_Text, F.Cu at (102.0, 117.0)
- moved LG1 310.6 mm to (375.0, 184.0)
- moved J1 0.50 mm to (60.0, 150.2)
Routing:
- net GND: track 15.6 -> 313.2 mm, vias 23 -> 295
- net /LED: track 21.7 -> 135.3 mm
- net /D+: track 12.2 -> 14.8 mm
- net /~{RESET}: track 83.9 -> 83.4 mm
- net /PGMR_SCK: track 43.0 -> 42.5 mm
- net /PGMR_MOSI: track 39.4 -> 38.9 mm
Other:
- board text added: "Revision 2.0 Sign Designed by: Kyle Schmerge"
- board text added: "UCSB IEEE Lab For Makers & Engineers ucsbieee.org"

Commit message: Update ieee-sign.kicad_pcb
Other:
- board text added: "+5V"
- board text added: "CC1"
- board text added: "CC2"
- board text added: "GND"
- board text added: "LED Signal"
- board text added: "Mode"
- board text added: "Reset"
Changed lines of the file:
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@@
 		(layer "Edge.Cuts")
+	)
+	(gr_text "CC1"
+		(at 56.5 164.25 0)
+		(layer "F.SilkS")
+		(effects
+			(font
+				(size 1 1)
+				(thickness 0.1)
+			)
+			(justify bottom)
+		)
+	)
+	(gr_text "CC2"
+		(at 56.5 168.25 0)
+		(layer "F.SilkS")
+		(effects
+			(font
+				(size 1 1)
+				(thickness 0.1)
+			)
+			(justify bottom)
+		)
+	)
+	(gr_text "+5V"
+		(at 81.1 154.3 0)
+		(layer "F.SilkS")
+		(effects
+			(font
+				(size 1 1)
+				(thickness 0.1)
+			)
+			(justify bottom)
+		)
+	)
+	(gr_text "GND"
+		(at 87.15 154.3 0)
+		(layer "F.SilkS")
+		(effects
+			(font
+				(size 1 1)
+				(thickness 0.1)
+			)
+			(justify bottom)
+		)
+	)
+	(gr_text "LED Signal"
+		(at 92.25 174.9 0)
+		(layer "F.SilkS")
+		(effects
+			(font
+				(size 1 1)
+				(thickness 0.1)
+			)
+			(justify bottom)
+		)
+	)
+	(gr_text "Mode"
+		(at 89.4 147.2 90)
+		(layer "F.SilkS")
+		(effects
+			(font
+				(size 1 1)
+				(thickness 0.1)
+			)
+		)
+	)
+	(gr_text "Reset"
+		(at 94.2 185.4 90)
+		(layer "F.SilkS")
+		(effects
+			(font
+				(size 1 1)
+				(thickness 0.1)
+			)
+		)
 	)
 	(gr_text "Revision 2.0\nSign Designed by:\nKyle Schmerge"
